File: GlowLEDsPCB.kicad_pcb (KiCad board)
At the start: 2 copper layers, 10 x 250 mm, 43 parts, among them U1 Contact pads, U2 Contact pads

Commit message: increased pcb thickness and extended pads to edges
Other:
- board text added: "v1.0 beta 2"
- board text removed: "v1.0 beta 1"
Changed lines of the file:
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@@
 (kicad_pcb (version 20211014) (generator pcbnew)
   (general
-    (thickness 1.09)
+    (thickness 1.69)
   )
   (paper "A4" portrait)
@@
   (setup
     (stackup
-      (layer "F.SilkS" (type "Top Silk Screen"))
+      (layer "F.SilkS" (type "Top Silk Screen") (color "Black"))
       (layer "F.Paste" (type "Top Solder Paste"))
-      (layer "F.Mask" (type "Top Solder Mask") (thickness 0.01))
+      (layer "F.Mask" (type "Top Solder Mask") (color "White") (thickness 0.01))
       (layer "F.Cu" (type "copper") (thickness 0.035))
-      (layer "dielectric 1" (type "core") (thickness 1) (material "FR4") (epsilon_r 4.5) (loss_tangent 0.02))
+      (layer "dielectric 1" (type "core") (thickness 1.6) (material "FR4") (epsilon_r 4.5) (loss_tangent 0.02))
       (layer "B.Cu" (type "copper") (thickness 0.035))
-      (layer "B.Mask" (type "Bottom Solder Mask") (thickness 0.01))
+      (layer "B.Mask" (type "Bottom Solder Mask") (color "White") (thickness 0.01))
       (layer "B.Paste" (type "Bottom Solder Paste"))
-      (layer "B.SilkS" (type "Bottom Silk Screen"))
+      (layer "B.SilkS" (type "Bottom Silk Screen") (color "Black"))
       (copper_finish "HAL lead-free")
       (dielectric_constraints no)
@@
     (pad_to_mask_clearance 0)
     (pcbplotparams
-      (layerselection 0x0041008_7ffffffe)
+      (layerselection 0x0001008_7ffffffe)
       (disableapertmacros false)
       (usegerberextensions false)
@@
       (drillshape 0)
       (scaleselection 1)
-      (outputdirectory "PCB stencils/")
+      (outputdirectory "./")
     )
   )
@@
     )
     (fp_rect (start -5 -12.1412) (end 5 -2.159) (layer "F.Fab") (width 0.12) (fill none))
-    (pad "1" smd rect locked (at -3.8338 -0.0056) (size 1.6 2.8) (layers "F.Cu" "F.Mask")
+    (pad "1" smd rect locked (at -3.8338 -0.2056) (size 1.6 3.2) (layers "F.Cu" "F.Mask")
       (net 1 "+5V") (pinfunction "5V") (pintype "bidirectional"))
-    (pad "2" smd rect locked (at -1.334534 -0.0056) (size 2 2.8) (layers "F.Cu" "F.Mask")
+    (pad "2" smd rect locked (at -1.334534 -0.2056) (size 2 3.2) (layers "F.Cu" "F.Mask")
       (net 18 "Net-(D15-Pad2)") (pinfunction "Data") (pintype "bidirectional"))
-    (pad "3" smd rect locked (at 1.364732 -0.0056) (size 2 2.8) (layers "F.Cu" "F.Mask")
+    (pad "3" smd rect locked (at 1.364732 -0.2056) (size 2 3.2) (layers "F.Cu" "F.Mask")
       (net 2 "GND") (pinfunction "GND") (pintype "bidirectional"))
-    (pad "4" smd rect locked (at 3.864 -0.0056) (size 1.6 2.8) (layers "F.Cu" "F.Mask")
+    (pad "4" smd rect locked (at 3.864 -0.2056) (size 1.6 3.2) (layers "F.Cu" "F.Mask")
       (net 19 "BUTTON") (pinfunction "BUTTON") (pintype "bidirectional"))
   )
@@
     )
     (fp_rect (start -5 -12.1412) (end 5 -2.159) (layer "F.Fab") (width 0.12) (fill none))
-    (pad "1" smd rect locked (at -3.8338 -0.0056) (size 1.6 2.8) (layers "F.Cu" "F.Mask")
+    (pad "1" smd rect locked (at -3.8338 0.2056) (size 1.6 3.2) (layers "F.Cu" "F.Mask")
       (net 1 "+5V") (pinfunction "5V") (pintype "bidirectional"))
-    (pad "2" smd rect locked (at -1.334534 -0.0056) (size 2 2.8) (layers "F.Cu" "F.Mask")
+    (pad "2" smd rect locked (at -1.334534 0.2056) (size 2 3.2) (layers "F.Cu" "F.Mask")
       (net 4 "Net-(D1-Pad4)") (pinfunction "Data") (pintype "bidirectional"))
-    (pad "3" smd rect locked (at 1.364732 -0.0056) (size 2 2.8) (layers "F.Cu" "F.Mask")
+    (pad "3" smd rect locked (at 1.364732 0.2056) (size 2 3.2) (layers "F.Cu" "F.Mask")
       (net 2 "GND") (pinfunction "GND") (pintype "bidirectional"))
-    (pad "4" smd rect locked (at 3.864 -0.0056) (size 1.6 2.8) (layers "F.Cu" "F.Mask")
+    (pad "4" smd rect locked (at 3.864 0.2056) (size 1.6 3.2) (layers "F.Cu" "F.Mask")
       (net 19 "BUTTON") (pinfunction "BUTTON") (pintype "bidirectional"))
   )
@@
     (effects (font (size 1 1) (thickness 0.15)) (justify left mirror))
   )
-  (gr_text "v1.0 beta 1" (at 54.38 142.98 90) (layer "B.SilkS")
+  (gr_text "v1.0 beta 2" (at 54.38 142.98 90) (layer "B.SilkS")
     (effects (font (size 1 1) (thickness 0.15)) (justify mirror))
   )

Commit message: updated to release candidate 1
Parts:
- moved C1 3.83 mm to (48.4, 267.1), turned to 90 degrees
Routing:
- net +5V: track 53.8 -> 63.3 mm, vias 0 -> 4
- net GND: track 53.2 -> 58.7 mm, vias 32 -> 33
Other:
- board text added: "v1.0 RC1"
- board text removed: "v1.0 beta 2"
